File: Entrenador1-SchDoc.sch (KiCad schematic (older format))
At the start: 88 parts, among them CON1 BARREL_JACK, J11 CON8, J3 ICSP, J5 CON8, J6 CON8, J7 CON8, J9 3vias, P1 CONN_01X04, P2 CONN_01X04, P3 CONN_01X07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

Commit message: adición del BOM
Parts:
- C10, C9: value C -> 22pf
- C11: value CP -> 1uf
- C6: value ~ -> 10uf
- C7: value C -> 100nf
- C8: value CP -> 47uf
- D12: value D -> 1n4004
- RV1, RV2: value POT -> 10K lin
- Y2: value XTAL -> 20MHz
- gave numbers to parts that had none: 2
Changed lines of the file:
@@
 LIBS:contrib
 LIBS:valves
-LIBS:w_analog
 LIBS:cmos_ieee
 LIBS:microchip_pic18mcu
@@
 P 9100 5750
 F 0 "C6" H 8800 5800 60  0000 L BNN
-F 1 "~" H 9100 5750 60  0001 C CNN
+F 1 "10uf" H 8900 5750 60  0000 C CNN
 F 2 "libreria:CP_Radial_D6.3mm_P2.50mm" H 9100 5750 60  0001 C CNN
 F 3 "" H 9100 5750 60  0001 C CNN
@@
 U 1 1 5A3E7AC7
 P 11400 4200
-F 0 "RV1" H 11400 4120 50  0000 C CNN
-F 1 "POT" H 11400 4200 50  0000 C CNN
+F 0 "RV1" V 11450 3900 50  0000 C CNN
+F 1 "10K lin" V 11350 3950 50  0000 C CNN
 F 2 "libreria:Potentiometer_Omeg_PC16PU_Horizontal" H 11400 4200 50  0001 C CNN
 F 3 "" H 11400 4200 50  0000 C CNN
@@
 U 1 1 5A3E7E62
 P 11400 4900
-F 0 "RV2" H 11400 4820 50  0000 C CNN
-F 1 "POT" H 11400 4900 50  0000 C CNN
+F 0 "RV2" V 11400 4600 50  0000 C CNN
+F 1 "10K lin" V 11300 4650 50  0000 C CNN
 F 2 "libreria:Potentiometer_Omeg_PC16PU_Horizontal" H 11400 4900 50  0001 C CNN
 F 3 "" H 11400 4900 50  0000 C CNN
@@
 U 1 1 5A6062F8
 P 7900 8550
-F 0 "C11" H 7925 8650 50  0000 L CNN
-F 1 "CP" H 7925 8450 50  0000 L CNN
+F 0 "C11" H 8050 8550 50  0000 L CNN
+F 1 "1uf" H 8050 8450 50  0000 L CNN
 F 2 "libreria:CP_Radial_D5.0mm_P2.50mm" H 7938 8400 50  0001 C CNN
 F 3 "" H 7900 8550 50  0000 C CNN
@@
 U 1 1 5A60A3BD
 P 4000 7900
-F 0 "C7" H 4025 8000 50  0000 L CNN
-F 1 "C" H 4025 7800 50  0000 L CNN
+F 0 "C7" H 4150 7950 50  0000 L CNN
+F 1 "100nf" H 4150 7850 50  0000 L CNN
 F 2 "libreria:C_Disc_D5.0mm_W2.5mm_P2.50mm" H 4038 7750 50  0001 C CNN
 F 3 "" H 4000 7900 50  0000 C CNN
@@
 P 6250 4050
 F 0 "C8" H 6275 4150 50  0000 L CNN
-F 1 "CP" H 6275 3950 50  0000 L CNN
+F 1 "47uf" H 6275 3950 50  0000 L CNN
 F 2 "libreria:CP_Radial_D5.0mm_P2.50mm" H 6288 3900 50  0001 C CNN
 F 3 "" H 6250 4050 50  0000 C CNN
@@
 P 5050 3900
 F 0 "D12" H 5050 4000 50  0000 C CNN
-F 1 "D" H 5050 3800 50  0000 C CNN
+F 1 "1n4004" H 5050 3800 50  0000 C CNN
 F 2 "libreria:D_5W_P10.16mm_Horizontal" H 5050 3900 50  0001 C CNN
 F 3 "" H 5050 3900 50  0000 C CNN
@@
 P 7100 6250
 F 0 "C9" H 7125 6350 50  0000 L CNN
-F 1 "C" H 7125 6150 50  0000 L CNN
+F 1 "22pf" H 7125 6150 50  0000 L CNN
 F 2 "libreria:C_Disc_D5.0mm_W2.5mm_P2.50mm" H 7138 6100 50  0001 C CNN
 F 3 "" H 7100 6250 50  0000 C CNN
@@
 P 7600 6250
 F 0 "C10" H 7625 6350 50  0000 L CNN
-F 1 "C" H 7625 6150 50  0000 L CNN
+F 1 "22pf" H 7625 6150 50  0000 L CNN
 F 2 "libreria:C_Disc_D5.0mm_W2.5mm_P2.50mm" H 7638 6100 50  0001 C CNN
 F 3 "" H 7600 6250 50  0000 C CNN
@@
 P 7300 6000
 F 0 "Y2" H 7300 6200 60  0000 L BNN
-F 1 "XTAL" H 7200 6100 60  0000 L BNN
+F 1 "20MHz" H 7200 6100 60  0000 L BNN
 F 2 "libreria:Crystal_HC49-4H_Vertical" H 7300 6000 60  0001 C CNN
 F 3 "" H 7300 6000 60  0000 C CNN
@@
 P 7100 6450
 F 0 "#PWR031" H 7100 6200 50  0001 C CNN
-F 1 "GND" H 7100 6300 50  0000 C CNN
+F 1 "GND" H 7100 6300 50  0001 C CNN
 F 2 "" H 7100 6450 50  0000 C CNN
 F 3 "" H 7100 6450 50  0000 C CNN
@@
 $EndComp
 $Comp
-L CONN_01X04 P?
+L CONN_01X04 P9
 U 1 1 5A72322A
 P 2300 2750
-F 0 "P?" H 2300 3000 50  0000 C CNN
+F 0 "P9" H 2300 3000 50  0000 C CNN
 F 1 "CONN_01X04" V 2400 2750 50  0000 C CNN
 F 2 "libreria:Socket_Strip_Straight_1x04_Pitch2.54mm" H 2300 2750 50  0001 C CNN
@@
 $EndComp
 $Comp
-L CONN_01X04 P?
+L CONN_01X04 P10
 U 1 1 5A723EA4
 P 2300 3250
-F 0 "P?" H 2300 3500 50  0000 C CNN
+F 0 "P10" H 2300 3500 50  0000 C CNN
 F 1 "CONN_01X04" V 2400 3250 50  0000 C CNN
 F 2 "libreria:Socket_Strip_Straight_1x04_Pitch2.54mm" H 2300 3250 50  0001 C CNN
@@
 $EndComp
 $Comp
-L VDD #PWR?
+L VDD #PWR054
 U 1 1 5A724122
 P 2700 2550
-F 0 "#PWR?" H 2700 2400 50  0001 C CNN
+F 0 "#PWR054" H 2700 2400 50  0001 C CNN
 F 1 "VDD" H 2700 2700 50  0000 C CNN
 F 2 "" H 2700 2550 50  0000 C CNN
@@
 Connection ~ 2700 2800
 $Comp
-L GND #PWR?
+L GND #PWR055
 U 1 1 5A724E72
 P 3250 3450
-F 0 "#PWR?" H 3250 3200 50  0001 C CNN
+F 0 "#PWR055" H 3250 3200 50  0001 C CNN
 F 1 "GND" H 3250 3300 50  0000 C CNN
 F 2 "" H 3250 3450 50  0000 C CNN

Commit message: cambio de huellas transistores, ajuste de pistas según prototipo
Parts:
- Q1, Q2, Q3, Q4: footprint libreria:TO-92_Inline_Narrow_Oval -> TO_SOT_Packages_THT:TO-92_Molded_Narrow
Changed lines of the file:
@@
 F 0 "Q1" H 15800 2375 50  0000 L CNN
 F 1 "BC548" H 15800 2300 50  0000 L CNN
-F 2 "libreria:TO-92_Inline_Narrow_Oval" H 15550 2850 50  0001 L CIN
+F 2 "TO_SOT_Packages_THT:TO-92_Molded_Narrow" H 15550 2850 50  0001 L CIN
 F 3 "" H 15600 2300 50  0000 L CNN
 	1    15600 2300
@@
 F 0 "Q2" H 15850 3825 50  0000 L CNN
 F 1 "BC548" H 15850 3750 50  0000 L CNN
-F 2 "libreria:TO-92_Inline_Narrow_Oval" H 15650 4300 50  0001 L CIN
+F 2 "TO_SOT_Packages_THT:TO-92_Molded_Narrow" H 15650 4300 50  0001 L CIN
 F 3 "" H 15650 3750 50  0000 L CNN
 	1    15650 3750
@@
 F 0 "Q3" H 15850 5275 50  0000 L CNN
 F 1 "BC548" H 15850 5200 50  0000 L CNN
-F 2 "libreria:TO-92_Inline_Narrow_Oval" H 15650 5750 50  0001 L CIN
+F 2 "TO_SOT_Packages_THT:TO-92_Molded_Narrow" H 15650 5750 50  0001 L CIN
 F 3 "" H 15650 5200 50  0000 L CNN
 	1    15650 5200
@@
 F 0 "Q4" H 15850 6725 50  0000 L CNN
 F 1 "BC548" H 15850 6650 50  0000 L CNN
-F 2 "libreria:TO-92_Inline_Narrow_Oval" H 15650 7200 50  0001 L CIN
+F 2 "TO_SOT_Packages_THT:TO-92_Molded_Narrow" H 15650 7200 50  0001 L CIN
 F 3 "" H 15650 6650 50  0000 L CNN
 	1    15650 6650

Commit message: En base al prototipo, se replantean las posiciones de los elementos
Parts:
- removed CON1: BARREL_JACK, libreria:BARREL_JACK, symbol BARREL_JACK
- R10, R11, R12, R13, R14, R15, R16, R9: value 330 -> 180
- R17, R18, R19, R20: value 470 -> 1200
- R21, R22, R23, R24, R25, R26, R27, R28: value 470 -> 180
- R29, R30, R31, R32: value 1200 -> 10k
Changed lines of the file:
@@
 P 5800 2500
 F 0 "R9" V 5910 2370 60  0000 R TNN
-F 1 "330" V 5810 2370 60  0000 R TNN
+F 1 "180" V 5810 2370 60  0000 R TNN
 F 2 "libreria:R_Axial_DIN0207_L6.3mm_D2.5mm_P7.62mm_Horizontal" H 5810 2370 60  0001 C CNN
 F 3 "" H 5810 2370 60  0000 C CNN
@@
 P 6350 2500
 F 0 "R10" V 6460 2370 60  0000 R TNN
-F 1 "330" V 6360 2370 60  0000 R TNN
+F 1 "180" V 6360 2370 60  0000 R TNN
 F 2 "libreria:R_Axial_DIN0207_L6.3mm_D2.5mm_P7.62mm_Horizontal" H 6360 2370 60  0001 C CNN
 F 3 "" H 6360 2370 60  0000 C CNN
@@
 P 6900 2500
 F 0 "R11" V 7010 2370 60  0000 R TNN
-F 1 "330" V 6910 2370 60  0000 R TNN
+F 1 "180" V 6910 2370 60  0000 R TNN
 F 2 "libreria:R_Axial_DIN0207_L6.3mm_D2.5mm_P7.62mm_Horizontal" H 6910 2370 60  0001 C CNN
 F 3 "" H 6910 2370 60  0000 C CNN
@@
 P 7450 2500
 F 0 "R12" V 7550 2350 60  0000 R TNN
-F 1 "330" V 7460 2370 60  0000 R TNN
+F 1 "180" V 7460 2370 60  0000 R TNN
 F 2 "libreria:R_Axial_DIN0207_L6.3mm_D2.5mm_P7.62mm_Horizontal" H 7460 2370 60  0001 C CNN
 F 3 "" H 7460 2370 60  0000 C CNN
@@
 P 8000 2500
 F 0 "R13" V 8100 2350 60  0000 R TNN
-F 1 "330" V 8010 2370 60  0000 R TNN
+F 1 "180" V 8010 2370 60  0000 R TNN
 F 2 "libreria:R_Axial_DIN0207_L6.3mm_D2.5mm_P7.62mm_Horizontal" H 8010 2370 60  0001 C CNN
 F 3 "" H 8010 2370 60  0000 C CNN
@@
 P 8500 2500
 F 0 "R14" V 8600 2350 60  0000 R TNN
-F 1 "330" V 8510 2370 60  0000 R TNN
+F 1 "180" V 8510 2370 60  0000 R TNN
 F 2 "libreria:R_Axial_DIN0207_L6.3mm_D2.5mm_P7.62mm_Horizontal" H 8510 2370 60  0001 C CNN
 F 3 "" H 8510 2370 60  0000 C CNN
@@
 P 9000 2500
 F 0 "R15" V 9100 2350 60  0000 R TNN
-F 1 "330" V 9010 2370 60  0000 R TNN
+F 1 "180" V 9010 2370 60  0000 R TNN
 F 2 "libreria:R_Axial_DIN0207_L6.3mm_D2.5mm_P7.62mm_Horizontal" H 9010 2370 60  0001 C CNN
 F 3 "" H 9010 2370 60  0000 C CNN
@@
 P 5250 2500
 F 0 "R16" V 5360 2370 60  0000 R TNN
-F 1 "330" V 5260 2370 60  0000 R TNN
+F 1 "180" V 5260 2370 60  0000 R TNN
 F 2 "libreria:R_Axial_DIN0207_L6.3mm_D2.5mm_P7.62mm_Horizontal" H 5260 2370 60  0001 C CNN
 F 3 "" H 5260 2370 60  0000 C CNN
@@
 P 15800 2600
 F 0 "R17" V 15910 2470 60  0000 R TNN
-F 1 "470" V 15810 2470 60  0000 R TNN
+F 1 "1200" V 15810 2470 60  0000 R TNN
 F 2 "libreria:R_Axial_DIN0207_L6.3mm_D2.5mm_P7.62mm_Horizontal" H 15810 2470 60  0001 C CNN
 F 3 "" H 15810 2470 60  0000 C CNN
@@
 P 15850 4050
 F 0 "R18" V 15960 3920 60  0000 R TNN
-F 1 "470" V 15860 3920 60  0000 R TNN
+F 1 "1200" V 15860 3920 60  0000 R TNN
 F 2 "libreria:R_Axial_DIN0207_L6.3mm_D2.5mm_P7.62mm_Horizontal" H 15860 3920 60  0001 C CNN
 F 3 "" H 15860 3920 60  0000 C CNN
@@
 P 15850 5500
 F 0 "R19" V 15960 5370 60  0000 R TNN
-F 1 "470" V 15860 5370 60  0000 R TNN
+F 1 "1200" V 15860 5370 60  0000 R TNN
 F 2 "libreria:R_Axial_DIN0207_L6.3mm_D2.5mm_P7.62mm_Horizontal" H 15860 5370 60  0001 C CNN
 F 3 "" H 15860 5370 60  0000 C CNN
@@
 P 15850 6950
 F 0 "R20" V 15960 6820 60  0000 R TNN
-F 1 "470" V 15860 6820 60  0000 R TNN
+F 1 "1200" V 15860 6820 60  0000 R TNN
 F 2 "libreria:R_Axial_DIN0207_L6.3mm_D2.5mm_P7.62mm_Horizontal" H 15860 6820 60  0001 C CNN
 F 3 "" H 15860 6820 60  0000 C CNN
@@
 P 15200 7750
 F 0 "R21" H 15800 7700 60  0000 R TNN
-F 1 "470" H 16050 7700 60  0000 R TNN
+F 1 "180" H 16050 7700 60  0000 R TNN
 F 2 "libreria:R_Axial_DIN0207_L6.3mm_D2.5mm_P7.62mm_Horizontal" H 15210 7620 60  0001 C CNN
 F 3 "" H 15210 7620 60  0000 C CNN
@@
 P 15200 7850
 F 0 "R22" H 15800 7800 60  0000 R TNN
-F 1 "470" H 16050 7800 60  0000 R TNN
+F 1 "180" H 16050 7800 60  0000 R TNN
 F 2 "libreria:R_Axial_DIN0207_L6.3mm_D2.5mm_P7.62mm_Horizontal" H 15210 7720 60  0001 C CNN
 F 3 "" H 15210 7720 60  0000 C CNN
@@
 P 15200 7950
 F 0 "R23" H 15800 7900 60  0000 R TNN
-F 1 "470" H 16050 7900 60  0000 R TNN
+F 1 "180" H 16050 7900 60  0000 R TNN
 F 2 "libreria:R_Axial_DIN0207_L6.3mm_D2.5mm_P7.62mm_Horizontal" H 15210 7820 60  0001 C CNN
 F 3 "" H 15210 7820 60  0000 C CNN
@@
 P 15200 8050
 F 0 "R24" H 15800 8000 60  0000 R TNN
-F 1 "470" H 16050 8000 60  0000 R TNN
+F 1 "180" H 16050 8000 60  0000 R TNN
 F 2 "libreria:R_Axial_DIN0207_L6.3mm_D2.5mm_P7.62mm_Horizontal" H 15210 7920 60  0001 C CNN
 F 3 "" H 15210 7920 60  0000 C CNN
@@
 P 15200 8150
 F 0 "R25" H 15800 8100 60  0000 R TNN
-F 1 "470" H 16050 8100 60  0000 R TNN
+F 1 "180" H 16050 8100 60  0000 R TNN
 F 2 "libreria:R_Axial_DIN0207_L6.3mm_D2.5mm_P7.62mm_Horizontal" H 15210 8020 60  0001 C CNN
 F 3 "" H 15210 8020 60  0000 C CNN
@@
 P 15200 8250
 F 0 "R26" H 15800 8200 60  0000 R TNN
-F 1 "470" H 16050 8200 60  0000 R TNN
+F 1 "180" H 16050 8200 60  0000 R TNN
 F 2 "libreria:R_Axial_DIN0207_L6.3mm_D2.5mm_P7.62mm_Horizontal" H 15210 8120 60  0001 C CNN
 F 3 "" H 15210 8120 60  0000 C CNN
@@
 P 15200 8350
 F 0 "R27" H 15800 8300 60  0000 R TNN
-F 1 "470" H 16050 8300 60  0000 R TNN
+F 1 "180" H 16050 8300 60  0000 R TNN
 F 2 "libreria:R_Axial_DIN0207_L6.3mm_D2.5mm_P7.62mm_Horizontal" H 15210 8220 60  0001 C CNN
 F 3 "" H 15210 8220 60  0000 C CNN
@@
 P 15200 8450
 F 0 "R28" H 15800 8400 60  0000 R TNN
-F 1 "470" H 16050 8400 60  0000 R TNN
+F 1 "180" H 16050 8400 60  0000 R TNN
 F 2 "libreria:R_Axial_DIN0207_L6.3mm_D2.5mm_P7.62mm_Horizontal" H 15210 8320 60  0001 C CNN
 F 3 "" H 15210 8320 60  0000 C CNN
@@
 P 11600 6650
 F 0 "R29" V 11700 6500 60  0000 R TNN
-F 1 "1200" V 11610 6520 60  0000 R TNN
+F 1 "10k" V 11610 6520 60  0000 R TNN
 F 2 "libreria:R_Axial_DIN0207_L6.3mm_D2.5mm_P7.62mm_Horizontal" H 11610 6520 60  0001 C CNN
 F 3 "" H 11610 6520 60  0000 C CNN
@@
 P 11950 6650
 F 0 "R30" V 12050 6500 60  0000 R TNN
-F 1 "1200" V 11960 6520 60  0000 R TNN
+F 1 "10k" V 11960 6520 60  0000 R TNN
 F 2 "libreria:R_Axial_DIN0207_L6.3mm_D2.5mm_P7.62mm_Horizontal" H 11960 6520 60  0001 C CNN
 F 3 "" H 11960 6520 60  0000 C CNN
@@
 P 12300 6650
 F 0 "R31" V 12400 6500 60  0000 R TNN
-F 1 "1200" V 12310 6520 60  0000 R TNN
+F 1 "10k" V 12310 6520 60  0000 R TNN
 F 2 "libreria:R_Axial_DIN0207_L6.3mm_D2.5mm_P7.62mm_Horizontal" H 12310 6520 60  0001 C CNN
 F 3 "" H 12310 6520 60  0000 C CNN
@@
 P 12650 6650
 F 0 "R32" V 12750 6500 60  0000 R TNN
-F 1 "1200" V 12660 6520 60  0000 R TNN
+F 1 "10k" V 12660 6520 60  0000 R TNN
 F 2 "libreria:R_Axial_DIN0207_L6.3mm_D2.5mm_P7.62mm_Horizontal" H 12660 6520 60  0001 C CNN
 F 3 "" H 12660 6520 60  0000 C CNN
@@
 $EndComp
 $Comp
-L BARREL_JACK CON1
-U 1 1 5A60D55A
-P 4400 4000
-F 0 "CON1" H 4400 4250 50  0000 C CNN
-F 1 "BARREL_JACK" H 4400 3800 50  0000 C CNN
-F 2 "libreria:BARREL_JACK" H 4400 4000 50  0001 C CNN
-F 3 "" H 4400 4000 50  0000 C CNN
-	1    4400 4000
-	1    0    0    1
-$EndComp
-$Comp
