File: Entrenador1-SchDoc.sch (KiCad schematic (older format))
At the start: 88 parts, among them J11 CON8, J3 ICSP, J5 CON8, J6 CON8, J7 CON8, J9 3vias, P1 CONN_01X04, P10 CONN_01X04, P2 CONN_01X04, P3 CONN_01X05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

Commit message: Pequeños ajustes repecto de las capas de información en el PCB
Parts:
- D10, D11, D4, D5, D6, D7, D8, D9: symbol LED -> LED-RESCUE-Entrenador1-SchDoc-RESCUE-Entrenador1-SchDoc
- D2, D3: symbol LED-RESCUE-Entrenador1-SchDoc -> LED-RESCUE-Entrenador1-SchDoc-RESCUE-Entrenador1-SchDoc
- P6: symbol USB_B -> USB_B-RESCUE-Entrenador1-SchDoc
- RV1, RV2: symbol POT -> POT-RESCUE-Entrenador1-SchDoc
Connections:
- net GND: now also D2.2 (K), D3.2 (K)
- net at R3.1: now also D2.1 (A)
- net at R4.1: now also D3.1 (A)
Changed lines of the file:
@@
 $EndComp
 $Comp
-L LED-RESCUE-Entrenador1-SchDoc D2
+L LED-RESCUE-Entrenador1-SchDoc-RESCUE-Entrenador1-SchDoc D2
 U 1 1 5A368A16
 P 9900 8500
@@
 $EndComp
 $Comp
-L LED-RESCUE-Entrenador1-SchDoc D3
+L LED-RESCUE-Entrenador1-SchDoc-RESCUE-Entrenador1-SchDoc D3
 U 1 1 5A368A15
 P 10500 8500
@@
 $EndComp
 $Comp
-L POT RV1
+L POT-RESCUE-Entrenador1-SchDoc RV1
 U 1 1 5A3E7AC7
 P 11400 4200
@@
 $EndComp
 $Comp
-L POT RV2
+L POT-RESCUE-Entrenador1-SchDoc RV2
 U 1 1 5A3E7E62
 P 11400 4900
@@
 Boton4
 $Comp
-L LED D4
+L LED-RESCUE-Entrenador1-SchDoc-RESCUE-Entrenador1-SchDoc D4
 U 1 1 5A5AB091
-P 5350 2900
-F 0 "D4" H 5350 3000 50  0000 C CNN
-F 1 "LED" H 5350 2800 50  0000 C CNN
-F 2 "libreria:LED_D3.0mm" H 5350 2900 50  0001 C CNN
-F 3 "" H 5350 2900 50  0000 C CNN
-	1    5350 2900
+P 5450 2900
+F 0 "D4" H 5450 3000 50  0000 C CNN
+F 1 "LED" H 5450 2800 50  0000 C CNN
+F 2 "libreria:LED_D3.0mm" H 5450 2900 50  0001 C CNN
+F 3 "" H 5450 2900 50  0000 C CNN
+	1    5450 2900
 	0    1    1    0
 $EndComp
 $Comp
-L LED D5
+L LED-RESCUE-Entrenador1-SchDoc-RESCUE-Entrenador1-SchDoc D5
 U 1 1 5A5AB849
-P 5900 2900
-F 0 "D5" H 5900 3000 50  0000 C CNN
-F 1 "LED" H 5900 2800 50  0000 C CNN
-F 2 "libreria:LED_D3.0mm" H 5900 2900 50  0001 C CNN
-F 3 "" H 5900 2900 50  0000 C CNN
-	1    5900 2900
+P 6000 2900
+F 0 "D5" H 6000 3000 50  0000 C CNN
+F 1 "LED" H 6000 2800 50  0000 C CNN
+F 2 "libreria:LED_D3.0mm" H 6000 2900 50  0001 C CNN
+F 3 "" H 6000 2900 50  0000 C CNN
+	1    6000 2900
 	0    1    1    0
 $EndComp
 $Comp
-L LED D6
+L LED-RESCUE-Entrenador1-SchDoc-RESCUE-Entrenador1-SchDoc D6
 U 1 1 5A5AB963
-P 6450 2900
-F 0 "D6" H 6450 3000 50  0000 C CNN
-F 1 "LED" H 6450 2800 50  0000 C CNN
-F 2 "libreria:LED_D3.0mm" H 6450 2900 50  0001 C CNN
-F 3 "" H 6450 2900 50  0000 C CNN
-	1    6450 2900
+P 6550 2900
+F 0 "D6" H 6550 3000 50  0000 C CNN
+F 1 "LED" H 6550 2800 50  0000 C CNN
+F 2 "libreria:LED_D3.0mm" H 6550 2900 50  0001 C CNN
+F 3 "" H 6550 2900 50  0000 C CNN
+	1    6550 2900
 	0    1    1    0
 $EndComp
 $Comp
-L LED D7
+L LED-RESCUE-Entrenador1-SchDoc-RESCUE-Entrenador1-SchDoc D7
 U 1 1 5A5ABA90
-P 7000 2900
-F 0 "D7" H 7000 3000 50  0000 C CNN
-F 1 "LED" H 7000 2800 50  0000 C CNN
-F 2 "libreria:LED_D3.0mm" H 7000 2900 50  0001 C CNN
-F 3 "" H 7000 2900 50  0000 C CNN
-	1    7000 2900
+P 7100 2900
+F 0 "D7" H 7100 3000 50  0000 C CNN
+F 1 "LED" H 7100 2800 50  0000 C CNN
+F 2 "libreria:LED_D3.0mm" H 7100 2900 50  0001 C CNN
+F 3 "" H 7100 2900 50  0000 C CNN
+	1    7100 2900
 	0    1    1    0
 $EndComp
 $Comp
-L LED D8
+L LED-RESCUE-Entrenador1-SchDoc-RESCUE-Entrenador1-SchDoc D8
 U 1 1 5A5ABBB0
-P 7550 2900
-F 0 "D8" H 7550 3000 50  0000 C CNN
-F 1 "LED" H 7550 2800 50  0000 C CNN
-F 2 "libreria:LED_D3.0mm" H 7550 2900 50  0001 C CNN
-F 3 "" H 7550 2900 50  0000 C CNN
-	1    7550 2900
+P 7650 2900
+F 0 "D8" H 7650 3000 50  0000 C CNN
+F 1 "LED" H 7650 2800 50  0000 C CNN
+F 2 "libreria:LED_D3.0mm" H 7650 2900 50  0001 C CNN
+F 3 "" H 7650 2900 50  0000 C CNN
+	1    7650 2900
 	0    1    1    0
 $EndComp
 $Comp
-L LED D9
+L LED-RESCUE-Entrenador1-SchDoc-RESCUE-Entrenador1-SchDoc D9
 U 1 1 5A5ABCCF
-P 8100 2900
-F 0 "D9" H 8100 3000 50  0000 C CNN
-F 1 "LED" H 8100 2800 50  0000 C CNN
-F 2 "libreria:LED_D3.0mm" H 8100 2900 50  0001 C CNN
-F 3 "" H 8100 2900 50  0000 C CNN
-	1    8100 2900
+P 8200 2900
+F 0 "D9" H 8200 3000 50  0000 C CNN
+F 1 "LED" H 8200 2800 50  0000 C CNN
+F 2 "libreria:LED_D3.0mm" H 8200 2900 50  0001 C CNN
+F 3 "" H 8200 2900 50  0000 C CNN
+	1    8200 2900
 	0    1    1    0
 $EndComp
 $Comp
-L LED D10
+L LED-RESCUE-Entrenador1-SchDoc-RESCUE-Entrenador1-SchDoc D10
 U 1 1 5A5ABDFD
-P 8600 2900
-F 0 "D10" H 8600 3000 50  0000 C CNN
-F 1 "LED" H 8600 2800 50  0000 C CNN
-F 2 "libreria:LED_D3.0mm" H 8600 2900 50  0001 C CNN
-F 3 "" H 8600 2900 50  0000 C CNN
-	1    8600 2900
+P 8700 2900
+F 0 "D10" H 8700 3000 50  0000 C CNN
+F 1 "LED" H 8700 2800 50  0000 C CNN
+F 2 "libreria:LED_D3.0mm" H 8700 2900 50  0001 C CNN
+F 3 "" H 8700 2900 50  0000 C CNN
+	1    8700 2900
 	0    1    1    0
 $EndComp
 $Comp
-L LED D11
+L LED-RESCUE-Entrenador1-SchDoc-RESCUE-Entrenador1-SchDoc D11
 U 1 1 5A5ABF28
-P 9100 2900
-F 0 "D11" H 9100 3000 50  0000 C CNN
-F 1 "LED" H 9100 2800 50  0000 C CNN
-F 2 "libreria:LED_D3.0mm" H 9100 2900 50  0001 C CNN
-F 3 "" H 9100 2900 50  0000 C CNN
-	1    9100 2900
+P 9200 2900
+F 0 "D11" H 9200 3000 50  0000 C CNN
+F 1 "LED" H 9200 2800 50  0000 C CNN
+F 2 "libreria:LED_D3.0mm" H 9200 2900 50  0001 C CNN
+F 3 "" H 9200 2900 50  0000 C CNN
+	1    9200 2900
 	0    1    1    0
 $EndComp
@@
 Wire Wire Line
 	5350 2100 5350 2200
-Wire Wire Line
-	5350 3100 9550 3100
-Connection ~ 5900 3100
-Connection ~ 6450 3100
-Connection ~ 7000 3100
-Connection ~ 7550 3100
-Connection ~ 8100 3100
-Connection ~ 8600 3100
-Connection ~ 9100 3100
 Wire Wire Line
 	14000 8450 13900 8450
@@
 	7500 8200 7400 8200
 $Comp
-L USB_B P6
+L USB_B-RESCUE-Entrenador1-SchDoc P6
 U 1 1 5A5E6768
 P 8600 8000
@@
 $EndComp
 $Comp
-L GND #PWR014
-U 1 1 5A60FD43
-P 4900 4300
-F 0 "#PWR014" H 4900 4050 50  0001 C CNN
-F 1 "GND" H 4900 4150 50  0000 C CNN
-F 2 "" H 4900 4300 50  0000 C CNN
-F 3 "" H 4900 4300 50  0000 C CNN
-	1    4900 4300
-	1    0    0    -1
-$EndComp
-$Comp
 L GND #PWR015
 U 1 1 5A60FE65
@@
 	1    0    0    -1
 $EndComp
-Wire Wire Line
-	4900 4100 4900 4300
 Wire Wire Line
 	5700 4300 5700 4200
@@
 L VDD #PWR022
 U 1 1 5A661943
-P 9550 3100
-F 0 "#PWR022" H 9550 2950 50  0001 C CNN
-F 1 "VDD" H 9550 3250 50  0000 C CNN
-F 2 "" H 9550 3100 50  0000 C CNN
-F 3 "" H 9550 3100 50  0000 C CNN
-	1    9550 3100
+P 9450 3300
+F 0 "#PWR022" H 9450 3150 50  0001 C CNN
+F 1 "VDD" H 9450 3450 50  0000 C CNN
+F 2 "" H 9450 3300 50  0000 C CNN
+F 3 "" H 9450 3300 50  0000 C CNN
+	1    9450 3300
 	0    1    1    0
 $EndComp
@@
 	1    0    0    -1
 $EndComp
-Wire Wire Line
-	4700 3900 4900 3900
-Wire Wire Line
-	4700 4100 4900 4100
 $Comp
 L SPST S3
@@
 Wire Wire Line
 	5400 5350 5150 5350
+Wire Wire Line
+	5350 3200 9100 3200
+Connection ~ 5900 3200
+Connection ~ 6450 3200
+Connection ~ 7000 3200
+Connection ~ 7550 3200
+Connection ~ 8100 3200
+Connection ~ 8600 3200
+Wire Wire Line
+	9100 3200 9200 3300
+Wire Wire Line
+	9200 3300 9450 3300
+Connection ~ 9100 3200
+Wire Wire Line
+	4750 3900 4900 3900
 $EndSCHEMATC

Commit message: modified:   Entrenador1-SchDoc.net 	modified:   Entrenador1-SchDoc.sch  Untracked files: 	Entrenador1-SchDoc_4Display_en_uno.kicad_pcb 	Entrenador1-SchDoc_4Display_en_uno.kicad_pcb-bak
Parts:
- added U1: CC56-12EWA, Displays_7-Segment:CA56-12EWA, symbol CC56-12EWA
Connections:
- net labels added: +5VFuente, CC1, CC2, CC3, CC4
- wire segments 251 -> 263
