File: Entrenador1-SchDoc_4Display_en_uno.sch (KiCad schematic (older format))
At the start: 85 parts, among them J11 CON8, J3 ICSP, J5 CON8, J6 CON8, J7 CON8, J9 3vias, P1 CONN_01X04, P10 CONN_01X04, P2 CONN_01X04, P3 CONN_01X05, P4 CONN_01X04, P5 CONN_01X09, P6 USB_B, P7 CONN_01X02, P8 CONN_01X02, P9 CONN_01X04, Q1 BC548, Q2 BC548, Q3 BC548, Q4 BC548, U1 CC56-12EWA, U2 ULN2803, U3 4511, U4 LM7805, U5 PIC18(L)F4550-I/P, Y2 20MHz

Commit message: Changes to be committed: 	modified:   Entrenador1-SchDoc_4Display_en_uno-cache.lib 	modified:   Entrenador1-SchDoc_4Display_en_uno.kicad_pcb 	modified:   Entrenador1-SchDoc_4Display_en_uno.kicad_pcb-bak 	modified:   Entrenador1-SchDoc_4Display_en_uno.sch 	modified:   Entrenador1-SchDoc_4Display_en_uno.sch-bak
Parts:
- Q1, Q2, Q3, Q4: footprint libreria:TO-92_Molded_Narrow -> TO_SOT_Packages_THT:TO-92_Molded_Narrow
- R1, R17, R18, R19, R2, R20, R21, R22, R23, R24, R25, R26, R27, R28, R29, R3, R30, R31, R32, R4, R6, R7, R8: symbol Entrenador1-SchDoc-rescue:Res1 -> Device:R_US
- U1: footprint libreria:CA56-12EWA -> Displays_7-Segment:CA56-12EWA
- U4: footprint libreria:TO-220-3_Vertical -> TO-220
- U5: footprint libreria:DIP-40_W15.24mm_LongPads -> DIP40
Connections:
- net Boton3: now also R7.1; no longer R7.2
- net Boton4: now also R8.1; no longer R8.2
- net Disp1: now also R17.2; no longer R17.1
- net Disp2: now also R18.2; no longer R18.1
- net Disp3: now also R19.2; no longer R19.1
- net Disp4: now also R20.2; no longer R20.1
- net DisplayH: now also R28.2; no longer R28.1
- net Display_A: now also R29.1; no longer R29.2
- net Display_B: now also R30.1; no longer R30.2
- net Display_C: now also R31.1; no longer R31.2
- net Display_D: now also R32.1; no longer R32.2
- net GNDD: now also R29.2, R30.2, R31.2, R32.2; no longer R29.1, R30.1, R31.1, R32.1
- net MCRL: now also R1.2; no longer R1.1
- net RB4: now also R2.2; no longer R2.1
- net RD0: now also R3.1; no longer R3.2
- net RD1: now also R4.1; no longer R4.2
- net VDD: now also R1.1, R2.1, R7.2, R8.2; no longer R1.2, R2.2, R7.1, R8.1
- net a: now also R21.1; no longer R21.2
- net b: now also R22.1; no longer R22.2
- net c: now also R23.1; no longer R23.2
- net d: now also R24.1; no longer R24.2
- net e: now also R25.1; no longer R25.2
- net f: now also R26.1; no longer R26.2
- net g: now also R27.1; no longer R27.2
- net h: now also R28.1; no longer R28.2
- net at D2.1 (A): now also R3.2; no longer R3.1
- net at D3.1 (A): now also R4.2; no longer R4.1
- net at U3.10 (Qd): now also R24.2; no longer R24.1
- net at U3.11 (Qc): now also R23.2; no longer R23.1
- net at U3.12 (Qb): now also R22.2; no longer R22.1
- net at U3.13 (Qa): now also R21.2; no longer R21.1
- net at U3.14 (Qg): now also R27.2; no longer R27.1
- net at U3.15 (Qf): now also R26.2; no longer R26.1
- net at U3.9 (Qe): now also R25.2; no longer R25.1
- net at Q1.2 (B): now also R17.1; no longer R17.2
- net at Q2.2 (B): now also R18.1; no longer R18.2
- net at Q3.2 (B): now also R19.1; no longer R19.2
- net at Q4.2 (B): now also R20.1; no longer R20.2
Other:
- moved on the sheet: R1, R17, R18, R19, R2, R20, R21, R22, R23, R24, R25, R26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

Commit message: modified:   Entrenador1-SchDoc_4Display_en_uno-cache.lib 	modified:   Entrenador1-SchDoc_4Display_en_uno.kicad_pcb 	modified:   Entrenador1-SchDoc_4Display_en_uno.kicad_pcb-bak 	modified:   Entrenador1-SchDoc_4Display_en_uno.net 	modified:   Entrenador1-SchDoc_4Display_en_uno.sch 	modified:   Entrenador1-SchDoc_4Display_en_uno.sch-bak 	modified:   fp-info-cache 	renamed:    Entrenador1-SchDoc-cache.lib -> lib_sch/Entrenador1-SchDoc-cache.lib 	renamed:    Entrenador1-SchDoc-rescue.lib -> lib_sch/Entrenador1-SchDoc-rescue.lib 	new file:   lib_sch/Entrenador1-SchDoc_4Display_en_uno.bck 	new file:   lib_sch/Entrenador1-SchDoc_4Display_en_uno.dcm 	new file:   lib_sch/Entrenador1-SchDoc_4Display_en_uno.lib 	modified:   sym-lib-table
Parts:
- C10, C7, C9: symbol Device:C -> Entrenador1-SchDoc_4Display_en_uno:Device_C
- C11, C6, C8: symbol Device:CP -> Entrenador1-SchDoc_4Display_en_uno:Device_CP
- D1, D12: symbol Device:D -> Entrenador1-SchDoc_4Display_en_uno:Device_D
- D10, D11, D2, D3, D4, D5, D6, D7, D8, D9: symbol Entrenador1-SchDoc-rescue:LED-RESCUE-Entrenador1-SchDoc-RESCUE-Entrenador1-SchDoc -> Entrenador1-SchDoc_4Display_en_uno:Device_LED
- J11: value CON8 -> LEDS; symbol Entrenador1-SchDoc-rescue:CONN_01X08 -> Entrenador1-SchDoc_4Display_en_uno:conn_Conn_01x08
- J3: symbol Entrenador1-SchDoc-rescue:CONN_01X06 -> Entrenador1-SchDoc_4Display_en_uno:conn_Conn_01x06
- J5, J6, J7: symbol Entrenador1-SchDoc-rescue:CONN_01X08 -> Entrenador1-SchDoc_4Display_en_uno:conn_Conn_01x08
- J9: symbol Entrenador1-SchDoc-rescue:CONN_01X03 -> Entrenador1-SchDoc_4Display_en_uno:conn_Conn_01x03
- JP1: symbol Entrenador1-SchDoc-rescue:JUMPER3 -> Entrenador1-SchDoc_4Display_en_uno:Device_Jumper_NC_Dual
- P1: symbol Entrenador1-SchDoc-rescue:CONN_01X04 -> Entrenador1-SchDoc_4Display_en_uno:conn_Conn_01x04
- P10: value CONN_01X04 -> Negativo; symbol Entrenador1-SchDoc-rescue:CONN_01X04 -> Entrenador1-SchDoc_4Display_en_uno:conn_Conn_01x04
- P2: value CONN_01X04 -> DISPLAY; symbol Entrenador1-SchDoc-rescue:CONN_01X04 -> Entrenador1-SchDoc_4Display_en_uno:conn_Conn_01x04
- P3: symbol Entrenador1-SchDoc-rescue:CONN_01X05 -> Entrenador1-SchDoc_4Display_en_uno:conn_Conn_01x05
- P4: value CONN_01X04 -> BOTONES; symbol Entrenador1-SchDoc-rescue:CONN_01X04 -> Entrenador1-SchDoc_4Display_en_uno:conn_Conn_01x04
- P5: symbol Entrenador1-SchDoc-rescue:CONN_01X09 -> Entrenador1-SchDoc_4Display_en_uno:conn_Conn_01x09
- P6: symbol Entrenador1-SchDoc-rescue:USB_B-RESCUE-Entrenador1-SchDoc -> Entrenador1-SchDoc_4Display_en_uno:Connector_USB_B
- P7: value CONN_01X02 -> 12V; symbol Entrenador1-SchDoc-rescue:CONN_01X02 -> Entrenador1-SchDoc_4Display_en_uno:conn_Conn_01x02
- P8: value CONN_01X02 -> 5V; symbol Entrenador1-SchDoc-rescue:CONN_01X02 -> Entrenador1-SchDoc_4Display_en_uno:conn_Conn_01x02
- P9: value CONN_01X04 -> Positivo; symbol Entrenador1-SchDoc-rescue:CONN_01X04 -> Entrenador1-SchDoc_4Display_en_uno:conn_Conn_01x04
- Q1, Q2, Q3, Q4: footprint TO_SOT_Packages_THT:TO-92_Molded_Narrow -> libreria:TO-92_Molded_Narrow; symbol transistors:BC548 -> Entrenador1-SchDoc_4Display_en_uno:BC548
- R1, R10, R11, R12, R13, R14, R15, R16, R17, R18, R19, R2, R20, R21, R22, R23, R24, R25, R26, R27, R28, R29, R3, R30, R31, R32, R4, R5, R6, R7, R8, R9: symbol Device:R_US -> Entrenador1-SchDoc_4Display_en_uno:Device_R_US
- RV1, RV2: symbol Entrenador1-SchDoc-rescue:POT-RESCUE-Entrenador1-SchDoc -> Entrenador1-SchDoc_4Display_en_uno:Device_R_POT_US
- S1, S2, S3, S4, S5, S6: symbol Entrenador1-SchDoc-rescue:SPST -> Entrenador1-SchDoc_4Display_en_uno:Switch_SW_Push
- U1: footprint Displays_7-Segment:CA56-12EWA -> libreria:CA56-12EWA; symbol display:CC56-12EWA -> Entrenador1-SchDoc_4Display_en_uno:display_CC56-12EWA
- U2: symbol Entrenador1-SchDoc-rescue:ULN2803 -> Entrenador1-SchDoc_4Display_en_uno:Transistor_Array_ULN2803A
- U3: symbol cmos_ieee:4511 -> Entrenador1-SchDoc_4Display_en_uno:cmos_ieee_4511
- U4: footprint TO-220 -> libreria:TO-220-3_Vertical; symbol Entrenador1-SchDoc-rescue:LM7805CT -> Entrenador1-SchDoc_4Display_en_uno:regul_LM7805_TO220
- U5: footprint DIP40 -> libreria:DIP-40_W15.24mm_LongPads; symbol Entrenador1-SchDoc-rescue:PIC18(L)F4550-I_P -> Entrenador1-SchDoc_4Display_en_uno:MCU_Microchip_PIC18_PIC18F4550-IP
- Y2: symbol Entrenador1-SchDoc-rescue:XTAL -> Entrenador1-SchDoc_4Display_en_uno:Device_Crystal
Connections:
- net GND: now also D2.1 (K), D3.1 (K); no longer D2.2 (K), D3.2 (K)
- net MCRL: now also R1.1; no longer R1.2
- net RB4: now also R2.1; no longer R2.2
- net VDD: now also R1.2, R2.2; no longer R1.1, R2.1
- net at R3.2: now also D2.2 (A); no longer D2.1 (A)
- net at R4.2: now also D3.2 (A); no longer D3.1 (A)
- net +12VFuente: no longer names the net of D12.2 (A), P7.2 (Pin_2)
- no-connect marks 0 -> 1
Other:
- note added: "Control de displays 7 seg\n"
- note added: "Potenciómetros para proposito general"
- note added: "Puertos\n"
- note added: "Pull Down Entradas ABCD\n"
- note added: "Pulsadores de propo/sito general conectados a pull up\n"
- note added: "Pulsadores para reinicio y modo bootloader\n"
- moved on the sheet: C10, C11, C6, C7, C8, C9, D1, D12, JP1, Q1, Q2, Q3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

Commit message: Changes to be committed: 	new file:   "Documentaci\303\263n/2020/.~lock.ListaComponentes.csv#" 	modified:   "Documentaci\303\263n/2020/Armado.aux" 	modified:   "Documentaci\303\263n/2020/Armado.tex" 	new file:   "Documentaci\303\263n/2020/ListaComponentes.csv" 	modified:   "Documentaci\303\263n/2020/Principal.log" 	modified:   "Documentaci\303\263n/2020/Principal.pdf" 	modified:   "Documentaci\303\263n/2020/Principal.synctex.gz" 	modified:   "Documentaci\303\263n/2020/Principal.tex" 	modified:   "Documentaci\303\263n/2020/Principal.toc" 	new file:   "Documentaci\303\263n/2020/imagenes/ComponentesEntrenador.pdf" 	new file:   "Documentaci\303\263n/2020/imagenes/Entrenador1-SchDoc_4Display_en_uno.png" 	new file:   "Documentaci\303\263n/2020/imagenes/Entrenador1-SchDoc_4Display_en_uno_perspectiva.png" 	new file:   "Documentaci\303\263n/2020/imagenes/Entrenador1-SchDoc_4Display_en_uno_perspectiva2.png" 	new file:   "Documentaci\303\263n/2020/imagenes/EsquematicoEntrenador.pdf" 	new file:   "Documentaci\303\263n/2020/imagenes/PistasEntrenador.pdf" 	deleted:    "Documentaci\303\263n/Entrenador.png" 	deleted:    "Documentaci\303\263n/Entrenador1-SchDoc_4Display_en_uno v13.png" 	deleted:    "Documentaci\303\263n/Entrenador1-SchDoc_4Display_en_uno v13.tif" 	deleted:    "Documentaci\303\263n/Vista3D.png" 	new file:   Entrenador1-SchDoc_4Display_en_uno (2).csv 	new file:   Entrenador1-SchDoc_4Display_en_uno.csv 	modified:   Entrenador1-SchDoc_4Display_en_uno.kicad_pcb 	modified:   Entrenador1-SchDoc_4Display_en_uno.kicad_pcb-bak 	modified:   Entrenador1-SchDoc_4Display_en_uno.net 	modified:   Entrenador1-SchDoc_4Display_en_uno.pro 	modified:   Entrenador1-SchDoc_4Display_en_uno.sch 	modified:   Entrenador1-SchDoc_4Display_en_uno.sch-bak 	new file:   Entrenador1-SchDoc_4Display_en_uno.xml 	new file:   _autosave-Entrenador1-SchDoc_4Display_en_uno.kicad_pcb 	modified:   fp-info-cache
Connections:
- net VA1: now reaches P1.3 (Pin_3), RV1.2
- net VA2: now reaches P1.2 (Pin_2), RV2.2
Other:
- note added: "Acceso a alimentación y botones\n"
- note added: "Circuitos auxiliares placa Base\n"
- note added: "Conexionado del display de 4 digitos"
- note added: "Decodificacoioón BCD a 7 segmentos\n\n"
- note added: "Detalle del circuito del display placa Frente\n"
- note added: "Entradas de alimentación ambas placas\n"
- note added: "Leds Placa Frente\n"
- note added: "Leds de salida placa Base\n"
- note added: "Microcontrolador\n"
- note added: "Multiplexado de displays\n"
- note added: "Oscilador uControlador\n"
- note added: "Potenciómetros para proposito general placa Base\n"
- note added: "Puertos Placa Base\n"
- note removed: "Control de displays 7 seg\n"
- note removed: "Potenciómetros para proposito general"
- note removed: "Puertos\n"
- moved on the sheet: C10, C11, C7, C8, C9, D1, D12, D2, D3, J3, J9, JP1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

Commit message: Changes to be committed: 	new file:   Circuito2.sch 	deleted:    "Documentaci\303\263n/2020/.~lock.ListaComponentes.csv#" 	modified:   "Documentaci\303\263n/2020/Armado.aux" 	modified:   "Documentaci\303\263n/2020/Armado.tex" 	modified:   "Documentaci\303\263n/2020/Introduccion.aux" 	modified:   "Documentaci\303\263n/2020/Principal.aux" 	modified:   "Documentaci\303\263n/2020/Principal.log" 	modified:   "Documentaci\303\263n/2020/Principal.pdf" 	modified:   "Documentaci\303\263n/2020/Principal.synctex.gz" 	modified:   "Documentaci\303\263n/2020/Principal.tex" 	modified:   "Documentaci\303\263n/2020/Principal.toc" 	new file:   "Documentaci\303\263n/2020/imagenes/logo2.jpg" 	deleted:    Entrenador1-SchDoc.csv 	deleted:    Entrenador1-SchDoc_4Display_en_uno (2).csv 	deleted:    Entrenador1-SchDoc_4Display_en_uno.csv 	modified:   Entrenador1-SchDoc_4Display_en_uno.kicad_pcb 	modified:   Entrenador1-SchDoc_4Display_en_uno.kicad_pcb-bak 	modified:   Entrenador1-SchDoc_4Display_en_uno.pro 	modified:   Entrenador1-SchDoc_4Display_en_uno.sch 	modified:   Entrenador1-SchDoc_4Display_en_uno.sch-bak 	deleted:    Gabinete/Base.FCStd 	deleted:    Gabinete/Base.FCStd1 	deleted:    Gabinete/Base.step 	deleted:    Gabinete/Entrenador1-SchDoc.step 	deleted:    Gabinete/Entrenador1-SchDoc1.step 	deleted:    Gabinete/Entrenador1_SchDoc.FCStd1 	deleted:    Gabinete/PlanoGabinete.pdf 	deleted:    Gabinete/frente.FCStd 	deleted:    Gabinete/frente.FCStd1 	deleted:    Gabinete/frente1.step 	deleted:    ImagenesCapturadas/Entrenador1-SchDoc.jpg 	deleted:    ImagenesCapturadas/Entrenador1-SchDoc.png 	deleted:    ImagenesCapturadas/Entrenador1-SchDoc_4Display_en_uno.png 	deleted:    _autosave-Entrenador1-SchDoc_4Display_en_uno.kicad_pcb 	new file:   _autosave-file5E8BEFED.sch
Connections:
- net GND: no longer C10.2, C9.2
Other:
- note removed: "Oscilador uControlador\n"
- moved on the sheet: C10, C11, C6, C7, C8, C9, D1, D10, D11, D12, D2, D3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

Commit message: Changes to be committed: 	new file:   CAM/Entrenador2020.FlatPrj 	new file:   "Documentaci\303\263n/2020/CAM_AcrilicoEntrenador_2.nc" 	new file:   "Documentaci\303\263n/2020/CAM_AcrilicoEntrenador_3.nc" 	modified:   Entrenador1-SchDoc_4Display_en_uno-cache.lib 	modified:   Entrenador1-SchDoc_4Display_en_uno.kicad_pcb 	modified:   Entrenador1-SchDoc_4Display_en_uno.kicad_pcb-bak 	modified:   Entrenador1-SchDoc_4Display_en_uno.net 	modified:   Entrenador1-SchDoc_4Display_en_uno.sch 	modified:   Entrenador1-SchDoc_4Display_en_uno.sch-bak 	new file:   Film/Entrenador1-SchDoc_4Display_en_uno-B_Cu.gbr_panelized.svg 	new file:   Film/Entrenador1-SchDoc_4Display_en_uno-Edge_Cuts.gbr_panelized.svg 	new file:   GerberOutput/Entrenador1-SchDoc_4Display_en_uno-B_Cu.gbr 	new file:   GerberOutput/Entrenador1-SchDoc_4Display_en_uno-Edge_Cuts.gbr 	new file:   GerberOutput/Entrenador1-SchDoc_4Display_en_uno-drl.rpt 	new file:   GerberOutput/Entrenador1-SchDoc_4Display_en_uno-drl_map.gbr 	new file:   GerberOutput/Entrenador1-SchDoc_4Display_en_uno.drl 	modified:   fp-info-cache
Parts:
- added H1, H2, H3, H4, H5, H6, H7, H8: MountingHole, Mounting_Holes:MountingHole_3.2mm_M3, symbol Mechanical:MountingHole
Changed lines of the file:
@@
+	1    0    0    -1
+$EndComp
+$Comp
+L Mechanical:MountingHole H1
+U 1 1 5E420D65
+P 7000 8300
+F 0 "H1" H 7100 8300 50  0000 L CNN
+F 1 "MountingHole" H 7100 8255 50  0001 L CNN
+F 2 "Mounting_Holes:MountingHole_3.2mm_M3" H 7000 8300 50  0001 C CNN
+F 3 "~" H 7000 8300 50  0001 C CNN
+	1    7000 8300
+	1    0    0    -1
+$EndComp
+$Comp
+L Mechanical:MountingHole H3
+U 1 1 5E465542
+P 7400 8300
+F 0 "H3" H 7500 8300 50  0000 L CNN
+F 1 "MountingHole" H 7500 8255 50  0001 L CNN
+F 2 "Mounting_Holes:MountingHole_3.2mm_M3" H 7400 8300 50  0001 C CNN
+F 3 "~" H 7400 8300 50  0001 C CNN
+	1    7400 8300
+	1    0    0    -1
+$EndComp
+$Comp
+L Mechanical:MountingHole H5
+U 1 1 5E46573D
+P 7800 8300
+F 0 "H5" H 7900 8300 50  0000 L CNN
+F 1 "MountingHole" H 7900 8255 50  0001 L CNN
+F 2 "Mounting_Holes:MountingHole_3.2mm_M3" H 7800 8300 50  0001 C CNN
+F 3 "~" H 7800 8300 50  0001 C CNN
+	1    7800 8300
+	1    0    0    -1
+$EndComp
+$Comp
+L Mechanical:MountingHole H7
+U 1 1 5E465A03
+P 8150 8300
+F 0 "H7" H 8250 8300 50  0000 L CNN
+F 1 "MountingHole" H 8250 8255 50  0001 L CNN
+F 2 "Mounting_Holes:MountingHole_3.2mm_M3" H 8150 8300 50  0001 C CNN
+F 3 "~" H 8150 8300 50  0001 C CNN
+	1    8150 8300
+	1    0    0    -1
+$EndComp
+$Comp
+L Mechanical:MountingHole H2
+U 1 1 5E465C78
+P 7000 8650
+F 0 "H2" H 7100 8650 50  0000 L CNN
+F 1 "MountingHole" H 7100 8605 50  0001 L CNN
+F 2 "Mounting_Holes:MountingHole_3.2mm_M3" H 7000 8650 50  0001 C CNN
+F 3 "~" H 7000 8650 50  0001 C CNN
+	1    7000 8650
+	1    0    0    -1
+$EndComp
+$Comp
+L Mechanical:MountingHole H4
+U 1 1 5E465E98
+P 7400 8650
+F 0 "H4" H 7500 8650 50  0000 L CNN
+F 1 "MountingHole" H 7500 8605 50  0001 L CNN
+F 2 "Mounting_Holes:MountingHole_3.2mm_M3" H 7400 8650 50  0001 C CNN
+F 3 "~" H 7400 8650 50  0001 C CNN
+	1    7400 8650
+	1    0    0    -1
+$EndComp
+$Comp
+L Mechanical:MountingHole H6
+U 1 1 5E4660B7
+P 7800 8650
+F 0 "H6" H 7900 8650 50  0000 L CNN
+F 1 "MountingHole" H 7900 8605 50  0001 L CNN
+F 2 "Mounting_Holes:MountingHole_3.2mm_M3" H 7800 8650 50  0001 C CNN
+F 3 "~" H 7800 8650 50  0001 C CNN
+	1    7800 8650
+	1    0    0    -1
+$EndComp
+$Comp
+L Mechanical:MountingHole H8
+U 1 1 5E4662D7
+P 8150 8650
+F 0 "H8" H 8250 8650 50  0000 L CNN
+F 1 "MountingHole" H 8250 8605 50  0001 L CNN
+F 2 "Mounting_Holes:MountingHole_3.2mm_M3" H 8150 8650 50  0001 C CNN
+F 3 "~" H 8150 8650 50  0001 C CNN
+	1    8150 8650
 	1    0    0    -1
 $EndComp
